File: Audio_Mixer_PCB_schematic/_autosave-Audio_Mixer_PCB_schematic.kicad_sch (KiCad schematic)
At the start: 75 parts, among them J1 AudioJack3, J2 AudioJack3, J3 AudioJack3, U1 TL074, U2 TL074, U3 TL074, U4 TL074, U5 TL074

Commit message: part assembly
Parts:
- added D1: LED, symbol Device:LED
- added R36: 3.3k, symbol Device:R
- added SW1: SW_SPST, symbol Switch:SW_SPST
Connections:
- net +9V: now also R36.2, SW1.2 (B); no longer BT1.1 (+)
- net GND: now also D1.1 (K)
- new net: D1.2 (A), R36.1
- new net: BT1.1 (+), SW1.1 (A)
Other:
- moved on the sheet: BT1
